Commit message: TF Update for handles; now 'handle' refers to the UNROTATED handle and 'handle_rotated' refers to the rotated handle in sim.
This is to bring sim closer to hardware, wherein 'handle' refers to TF of the unrotated handle of the real device (defined by AprilTag).

File: manipulation_playground_articulated_devices/devices/DN40_globe_valve/model/DN40_globe_valve.urdf.xacro (robot description, xacro)
@@ -43,9 +43,15 @@
         </inertial>
     </link>
-    <!-- Globe Valve Joint -->
-    <joint name="globe_valve_joint" type="continuous">
+    <joint name="globe_valve_handle_to_base" type="fixed">
         <parent link="base"/>
         <child link="handle"/>
         <origin xyz="0 0 0.325" rpy="0 0 0"/>
+    </joint>
+    <link name="handle"/>
+    <!-- Globe Valve Joint -->
+    <joint name="globe_valve_joint" type="continuous">
+        <parent link="handle"/>
+        <child link="handle_rotated"/>
+        <origin xyz="0 0 0" rpy="0 0 0"/>
         <axis xyz="0 0 1"/>
         <dynamics damping="0.0" friction="10.0" />
@@ -63,5 +69,5 @@
     </transmission>
     <!-- Globe Valve Handle -->
-    <link name="handle">
+    <link name="handle_rotated">
         <collision>
             <origin xyz="0 0 0" rpy="0 0 0"/>

File: manipulation_playground_articulated_devices/devices/PN16_gate_valve/model/PN16_gate_valve.urdf.xacro (robot description, xacro)
@@ -23,7 +23,7 @@
     <link name="base">
         <collision>
-            <origin xyz="0 0 0" rpy="-1.5708 0 0"/>
+            <origin xyz="0 0 0.05" rpy="0 0 0"/>
             <geometry>
-                <mesh filename="package://manipulation_playground_articulated_devices/devices/PN16_gate_valve/model/PN16_gate_valve_base.dae"/>
+                <box size="0.13 0.13 0.24"/>
             </geometry>
         </collision>
@@ -43,8 +43,14 @@
         </inertial>
     </link>
-    <!-- Needle Valve Joint -->
-    <joint name="gate_valve_joint" type="continuous">
+    <joint name="gate_valve_handle_to_base" type="fixed">
         <parent link="base"/>
         <child link="handle"/>
+        <origin xyz="0 0 0.22" rpy="0 0 0"/>
+    </joint>
+    <link name="handle"/>
+    <!-- Gate Valve Joint -->
+    <joint name="gate_valve_joint" type="continuous">
+        <parent link="handle"/>
+        <child link="handle_rotated"/>
         <origin xyz="0 0 0" rpy="0 0 0"/>
         <axis xyz="0 0 1"/>
@@ -63,7 +69,7 @@
     </transmission>
     <!-- Gate Valve Handle -->
-    <link name="handle">
+    <link name="handle_rotated">
         <collision>
-            <origin xyz="0 0 0" rpy="-1.5708 0 0"/>
+            <origin xyz="0 0 -0.22" rpy="-1.5708 0 0"/>
             <geometry>
                 <mesh filename="package://manipulation_playground_articulated_devices/devices/PN16_gate_valve/model/PN16_gate_valve_handle.dae"/>
@@ -71,5 +77,5 @@
         </collision>
         <visual>
-            <origin xyz="0 0 0" rpy="-1.5708 0 0"/>
+            <origin xyz="0 0 -0.22" rpy="-1.5708 0 0"/>
             <geometry>
                 <mesh filename="package://manipulation_playground_articulated_devices/devices/PN16_gate_valve/model/PN16_gate_valve_handle.dae"/>
@@ -77,5 +83,5 @@
         </visual>
         <inertial>
-            <origin xyz="0 0 0" rpy="-1.5708 0 0"/>
+            <origin xyz="0 0 -0.22" rpy="-1.5708 0 0"/>
             <mass value="${mass2}"/>
             <inertia

File: manipulation_playground_articulated_devices/devices/VDL_6_20_110_ball_valve/model/VDL_6_20_110_ball_valve.urdf.xacro (robot description, xacro)
@@ -43,9 +43,15 @@
         </inertial>
     </link>
+    <joint name="ball_valve_handle_to_base" type="fixed">
+        <parent link="base"/>
+        <child link="handle"/>
+        <origin xyz="0 0 0.145" rpy="0 0 0"/>
+    </joint>
+    <link name="handle"/>
     <!-- Ball Valve Joint -->
     <joint name="ball_valve_joint" type="revolute">
-        <parent link="base"/>
-        <child link="handle"/>
-        <origin xyz="0 0 0.15" rpy="0 0 0"/>
+        <parent link="handle"/>
+        <child link="handle_rotated"/>
+        <origin xyz="0 0 0" rpy="0 0 0"/>
         <axis xyz="0 0 1"/>
         <dynamics damping="0.0" friction="10.0" />
@@ -63,5 +69,5 @@
     </transmission>
     <!-- Ball Valve Handle -->
-    <link name="handle">
+    <link name="handle_rotated">
         <collision>
             <origin xyz="0 0 -0.145" rpy="0 0 0"/>

File: manipulation_playground_articulated_devices/devices/needle_valve/model/needle_valve.urdf.xacro (robot description, xacro)
@@ -43,9 +43,15 @@
         </inertial>
     </link>
+    <joint name="needle_valve_handle_to_base" type="fixed">
+        <parent link="base"/>
+        <child link="handle"/>
+        <origin xyz="0 0 0.071" rpy="0 0 0"/>
+    </joint>
+    <link name="handle"/>
     <!-- Needle Valve Joint -->
     <joint name="needle_valve_joint" type="continuous">
-        <parent link="base"/>
-        <child link="handle"/>
-        <origin xyz="0 0 0.071" rpy="0 0 0"/> <!-- 0.071 -->
+        <parent link="handle"/>
+        <child link="handle_rotated"/>
+        <origin xyz="0 0 0" rpy="0 0 0"/>
         <axis xyz="0 0 1"/>
         <dynamics damping="0.0" friction="0.01" />
@@ -62,7 +68,7 @@
     </transmission>
     <!-- Needle Valve Handle -->
-    <link name="handle">
+    <link name="handle_rotated">
         <collision>
-            <origin xyz="0 0 0" rpy="0 -1.5708 0"/>
+            <origin xyz="0 0 0" rpy="0 -1.5708 1.5708"/>
             <geometry>
                 <cylinder radius="0.0063" length="0.055"/>
@@ -70,5 +76,5 @@
         </collision>
         <visual>
-            <origin xyz="0 0 -0.071" rpy="-1.5708 0 -1.5708"/>
+            <origin xyz="0 0 -0.071" rpy="-1.5708 0 0"/>
             <geometry>
                 <mesh filename="package://manipulation_playground_articulated_devices/devices/needle_valve/model/needle_valve_handle.dae"/>

Commit message: Added inertias to virtual 'handle' links to allow aimulation in Gazebo

File: manipulation_playground_articulated_devices/devices/DN40_globe_valve/model/DN40_globe_valve.urdf.xacro (robot description, xacro)
@@ -48,5 +48,14 @@
         <origin xyz="0 0 0.325" rpy="0 0 0"/>
     </joint>
-    <link name="handle"/>
+    <link name="handle">
+        <inertial>
+            <origin xyz="0 0 0" rpy="0 0 0" />
+            <mass value="1" />
+            <inertia
+            ixx="1.0" ixy="0.0" ixz="0.0"
+            iyy="1.0" iyz="0.0"
+            izz="1.0" />
+        </inertial>
+    </link>
     <!-- Globe Valve Joint -->
     <joint name="globe_valve_joint" type="continuous">

File: manipulation_playground_articulated_devices/devices/PN16_gate_valve/model/PN16_gate_valve.urdf.xacro (robot description, xacro)
@@ -48,5 +48,14 @@
         <origin xyz="0 0 0.22" rpy="0 0 0"/>
     </joint>
-    <link name="handle"/>
+    <link name="handle">
+        <inertial>
+            <origin xyz="0 0 0" rpy="0 0 0" />
+            <mass value="1" />
+            <inertia
+            ixx="1.0" ixy="0.0" ixz="0.0"
+            iyy="1.0" iyz="0.0"
+            izz="1.0" />
+        </inertial>
+    </link>
     <!-- Gate Valve Joint -->
     <joint name="gate_valve_joint" type="continuous">

File: manipulation_playground_articulated_devices/devices/VDL_6_20_110_ball_valve/model/VDL_6_20_110_ball_valve.urdf.xacro (robot description, xacro)
@@ -48,5 +48,14 @@
         <origin xyz="0 0 0.145" rpy="0 0 0"/>
     </joint>
-    <link name="handle"/>
+    <link name="handle">
+        <inertial>
+            <origin xyz="0 0 0" rpy="0 0 0" />
+            <mass value="1" />
+            <inertia
+            ixx="1.0" ixy="0.0" ixz="0.0"
+            iyy="1.0" iyz="0.0"
+            izz="1.0" />
+        </inertial>
+    </link>
     <!-- Ball Valve Joint -->
     <joint name="ball_valve_joint" type="revolute">

File: manipulation_playground_articulated_devices/devices/needle_valve/model/needle_valve.urdf.xacro (robot description, xacro)
@@ -48,5 +48,14 @@
         <origin xyz="0 0 0.071" rpy="0 0 0"/>
     </joint>
-    <link name="handle"/>
+    <link name="handle">
+        <inertial>
+            <origin xyz="0 0 0" rpy="0 0 0" />
+            <mass value="1" />
+            <inertia
+            ixx="1.0" ixy="0.0" ixz="0.0"
+            iyy="1.0" iyz="0.0"
+            izz="1.0" />
+        </inertial>
+    </link>
     <!-- Needle Valve Joint -->
     <joint name="needle_valve_joint" type="continuous">
