Commit message: Renamed 'handle' device to 'valve'

File: manipulation_playground_articulated_devices/devices/valve/model/valve.urdf.xacro (robot description, xacro)
@@ -1,8 +1,8 @@
 <?xml version="1.0"?>
-<!-- Interactable Handle -->
-<robot name="handle" xmlns:xacro="http://www.ros.org/wiki/xacro">
+<!-- Interactable Valve -->
+<robot name="valve" xmlns:xacro="http://www.ros.org/wiki/xacro">
     <xacro:arg name="continuous" default="true"/>
-    <xacro:macro name="handle" params="continuous:=true">
-        <!-- Constants for Handle Dimensions -->
+    <xacro:macro name="valve" params="continuous:=true">
+        <!-- Constants for Valve Dimensions -->
         <!-- Base -->
         <xacro:property name="width" value="0.1"/>
@@ -23,15 +23,15 @@
         <xacro:property name="grip_offset_from_edge" value="0.016"/>
         <!-- Import all Gazebo-customization elements, including Gazebo colors -->
-        <xacro:include filename="$(find manipulation_playground_articulated_devices)/devices/handle/model/handle.gazebo" />
+        <xacro:include filename="$(find manipulation_playground_articulated_devices)/devices/valve/model/valve.gazebo" />
         <!-- Import Rviz colors -->
-        <xacro:include filename="$(find manipulation_playground_articulated_devices)/devices/handle/model/materials.xacro" />
+        <xacro:include filename="$(find manipulation_playground_articulated_devices)/devices/valve/model/materials.xacro" />
         <!-- Used to fix device to world -->
         <link name="world"/>
-        <joint name="handle_base_to_world" type="fixed">
+        <joint name="valve_base_to_world" type="fixed">
             <parent link="world"/>
             <child link="base"/>
             <origin xyz="0 0 0" rpy="0 0 0"/>
         </joint>
-        <!-- Handle Base -->
+        <!-- Valve Base -->
         <link name="base">
             <collision>
@@ -57,5 +57,5 @@
             </inertial>
         </link>
-        <joint name="handle_handle_to_base" type="fixed">
+        <joint name="valve_handle_to_base" type="fixed">
             <parent link="base"/>
             <child link="handle"/>
@@ -72,7 +72,7 @@
             </inertial>
         </link>
-        <!-- Handle Joint -->
+        <!-- Valve Joint -->
         <xacro:if value="${continuous}">
-            <joint name="handle_joint" type="continuous">
+            <joint name="valve_joint" type="continuous">
                 <parent link="handle"/>
                 <child link="handle_rotated"/>
@@ -84,5 +84,5 @@
         </xacro:if>
         <xacro:unless value="${continuous}">
-            <joint name="handle_joint" type="revolute">
+            <joint name="valve_joint" type="revolute">
                 <parent link="handle"/>
                 <child link="handle_rotated"/>
@@ -93,15 +93,15 @@
             </joint>
         </xacro:unless>
-        <transmission name="handle_trans">
+        <transmission name="valve_trans">
             <type>transmission_interface/SimpleTransmission</type>
-            <joint name="handle_joint">
+            <joint name="valve_joint">
                 <hardwareInterface>hardware_interface/EffortJointInterface</hardwareInterface>
             </joint>
-            <actuator name="handle_actuator">
+            <actuator name="valve_actuator">
                 <hardwareInterface>hardware_interface/EffortJointInterface</hardwareInterface>
                 <mechanicalReduction>1</mechanicalReduction>
             </actuator>
         </transmission>
-        <!-- Handle Neck -->
+        <!-- Valve Handle Neck -->
         <link name="handle_rotated">
             <collision>
@@ -132,5 +132,5 @@
             <origin xyz="0 0 ${length2}" rpy="0 0 0"/>
         </joint>
-        <!-- Handle Ring -->
+        <!-- Valve Handle Ring -->
         <link name="ring">
             <collision>
@@ -156,6 +156,6 @@
             </inertial>
         </link>
-        <!-- Handle Grip Joint -->
-        <joint name="handle_ring_to_grip" type="fixed">
+        <!-- Valve Handle Grip Joint -->
+        <joint name="valve_ring_to_grip" type="fixed">
             <parent link="ring"/>
             <child link="grip"/>
@@ -165,5 +165,5 @@
             <limit effort="100" velocity="10" /> -->
         </joint>
-        <!-- Handle Grip -->
+        <!-- Valve Handle Grip -->
         <link name="grip">
             <collision>
@@ -190,4 +190,4 @@
         </link>
     </xacro:macro>
-    <xacro:handle continuous="$(arg continuous)"/>
+    <xacro:valve continuous="$(arg continuous)"/>
 </robot>
