Commit message: Added DN40_globe_valve and VDL_6_20_110_ball_valve.
Changed the orientation of PN16_gate_valve to match the standard with other devices.

Fixed broken TF for HNF361_safety_switch.

File: manipulation_playground_articulated_devices/devices/HNF361_safety_switch/model/HNF361_safety_switch.urdf.xacro (robot description, xacro)
@@ -23,5 +23,5 @@
     <link name="base">
         <collision>
-            <origin xyz="0 0 0" rpy="0 0 0"/>
+            <origin xyz="0 0 0" rpy="-1.5708 0 0"/>
             <geometry>
                 <mesh filename="package://manipulation_playground_articulated_devices/devices/HNF361_safety_switch/model/HNF361_safety_switch_base.dae"/>
@@ -29,5 +29,5 @@
         </collision>
         <visual>
-            <origin xyz="0 0 0" rpy="0 0 0"/>
+            <origin xyz="0 0 0" rpy="-1.5708 0 0"/>
             <geometry>
                 <mesh filename="package://manipulation_playground_articulated_devices/devices/HNF361_safety_switch/model/HNF361_safety_switch_base.dae"/>
@@ -35,5 +35,5 @@
         </visual>
         <inertial>
-            <origin xyz="0 0 ${height1/2}" rpy="0 0 0"/>
+            <origin xyz="0 0 ${height1/2}" rpy="-1.5708 0 0"/>
             <mass value="${mass1}"/>
             <inertia
@@ -49,5 +49,5 @@
         <origin xyz="0 -0.043 0.015" rpy="0 0 0"/>
         <axis xyz="1 0 0"/>
-        <dynamics damping="0.0" friction="0.0" />
+        <dynamics damping="0.0" friction="10.0" />
         <limit effort="100" lower="-1.5707" upper="0" velocity="0.5" />
     </joint>
@@ -65,5 +65,5 @@
     <link name="lever">
         <collision>
-            <origin xyz="0 0.043 -0.015" rpy="0 0 0"/>
+            <origin xyz="0 0.043 -0.015" rpy="-1.5708 0 0"/>
             <geometry>
                 <mesh filename="package://manipulation_playground_articulated_devices/devices/HNF361_safety_switch/model/HNF361_safety_switch_lever.dae"/>
@@ -71,5 +71,5 @@
         </collision>
         <visual>
-            <origin xyz="0 0.043 -0.015" rpy="0 0 0"/>
+            <origin xyz="0 0.043 -0.015" rpy="-1.5708 0 0"/>
             <geometry>
                 <mesh filename="package://manipulation_playground_articulated_devices/devices/HNF361_safety_switch/model/HNF361_safety_switch_lever.dae"/>
@@ -77,5 +77,5 @@
         </visual>
         <inertial>
-            <origin xyz="0 0 0" rpy="0 0 0"/>
+            <origin xyz="0 0 0" rpy="-1.5708 0 0"/>
             <mass value="${mass2}"/>
             <inertia

File: manipulation_playground_articulated_devices/devices/PN16_gate_valve/model/PN16_gate_valve.urdf.xacro (robot description, xacro)
@@ -23,5 +23,5 @@
     <link name="base">
         <collision>
-            <origin xyz="0 0 0" rpy="0 0 0"/>
+            <origin xyz="0 0 0" rpy="-1.5708 0 0"/>
             <geometry>
                 <mesh filename="package://manipulation_playground_articulated_devices/devices/PN16_gate_valve/model/PN16_gate_valve_base.dae"/>
@@ -29,5 +29,5 @@
         </collision>
         <visual>
-            <origin xyz="0 0 0" rpy="0 0 0"/>
+            <origin xyz="0 0 0" rpy="-1.5708 0 0"/>
             <geometry>
                 <mesh filename="package://manipulation_playground_articulated_devices/devices/PN16_gate_valve/model/PN16_gate_valve_base.dae"/>
@@ -35,5 +35,5 @@
         </visual>
         <inertial>
-            <origin xyz="0 0 ${height1/2}" rpy="0 0 0"/>
+            <origin xyz="0 0 ${height1/2}" rpy="-1.5708 0 0"/>
             <mass value="${mass1}"/>
             <inertia
@@ -48,5 +48,5 @@
         <child link="handle"/>
         <origin xyz="0 0 0" rpy="0 0 0"/>
-        <axis xyz="0 1 0"/>
+        <axis xyz="0 0 1"/>
         <dynamics damping="0.0" friction="10.0" />
         <limit effort="100" velocity="0.5" />
@@ -65,5 +65,5 @@
     <link name="handle">
         <collision>
-            <origin xyz="0 0 0" rpy="0 0 0"/>
+            <origin xyz="0 0 0" rpy="-1.5708 0 0"/>
             <geometry>
                 <mesh filename="package://manipulation_playground_articulated_devices/devices/PN16_gate_valve/model/PN16_gate_valve_handle.dae"/>
@@ -71,5 +71,5 @@
         </collision>
         <visual>
-            <origin xyz="0 0 0" rpy="0 0 0"/>
+            <origin xyz="0 0 0" rpy="-1.5708 0 0"/>
             <geometry>
                 <mesh filename="package://manipulation_playground_articulated_devices/devices/PN16_gate_valve/model/PN16_gate_valve_handle.dae"/>
@@ -77,5 +77,5 @@
         </visual>
         <inertial>
-            <origin xyz="0 0 0" rpy="0 0 0"/>
+            <origin xyz="0 0 0" rpy="-1.5708 0 0"/>
             <mass value="${mass2}"/>
             <inertia

Commit message: Minor fixes

File: manipulation_playground_articulated_devices/devices/HNF361_safety_switch/model/HNF361_safety_switch.urdf.xacro (robot description, xacro)
@@ -48,7 +48,7 @@
             <parent link="base"/>
             <child link="lever"/>
-            <origin xyz="0 -0.043 0.015" rpy="0 0 0"/>
+            <origin xyz="0 0.011 0.045" rpy="0 0 0"/>
             <axis xyz="1 0 0"/>
-            <dynamics damping="0.0" friction="10.0" />
+            <dynamics damping="0.0" friction="0.01" />
             <limit effort="100" lower="-1.5707" upper="0" velocity="0.5" />
         </joint>
@@ -66,5 +66,5 @@
         <link name="lever">
             <collision>
-                <origin xyz="0 0.043 -0.015" rpy="-1.5708 0 0"/>
+                <origin xyz="0 -0.011 -0.045" rpy="-1.5708 0 0"/>
                 <geometry>
                     <mesh filename="package://manipulation_playground_articulated_devices/devices/HNF361_safety_switch/model/HNF361_safety_switch_lever.dae"/>
@@ -72,5 +72,5 @@
             </collision>
             <visual>
-                <origin xyz="0 0.043 -0.015" rpy="-1.5708 0 0"/>
+                <origin xyz="0 -0.011 -0.045" rpy="-1.5708 0 0"/>
                 <geometry>
                     <mesh filename="package://manipulation_playground_articulated_devices/devices/HNF361_safety_switch/model/HNF361_safety_switch_lever.dae"/>

File: manipulation_playground_articulated_devices/devices/VDL_6_20_110_ball_valve/model/VDL_6_20_110_ball_valve.urdf.xacro (robot description, xacro)
@@ -65,5 +65,5 @@
             <origin xyz="0 0 0" rpy="0 0 0"/>
             <axis xyz="0 0 1"/>
-            <dynamics damping="0.0" friction="10.0" />
+            <dynamics damping="0.0" friction="0.01" />
             <limit effort="100" velocity="0.5" lower="0" upper="1.5708" />
         </joint>
