Commit message: Updates to needle valve, launch file renaming

File: manipulation_playground_articulated_devices/devices/needle_valve/model/needle_valve.urdf.xacro (robot description, xacro)
@@ -10,5 +10,5 @@
     <xacro:property name="length2" value="0.01"/>
     <xacro:property name="radius2" value="0.03"/>
-    <xacro:property name="mass2" value="0.05"/>
+    <xacro:property name="mass2" value="1"/>
     <!-- Import all Gazebo-customization elements -->
     <xacro:include filename="$(find manipulation_playground_articulated_devices)/devices/needle_valve/model/needle_valve.gazebo" />
@@ -23,11 +23,11 @@
     <link name="base">
         <collision>
-            <origin xyz="0 0 0" rpy="0 0 0"/>
+            <origin xyz="0 0 0.01" rpy="-1.5708 0 -1.5708"/>
             <geometry>
-                <mesh filename="package://manipulation_playground_articulated_devices/devices/needle_valve/model/needle_valve_base.dae"/>
+                <box size="0.065 0.05 0.03"/>
             </geometry>
         </collision>
         <visual>
-            <origin xyz="0 0 0" rpy="0 0 0"/>
+            <origin xyz="0 0 0" rpy="-1.5708 0 -1.5708"/>
             <geometry>
                 <mesh filename="package://manipulation_playground_articulated_devices/devices/needle_valve/model/needle_valve_base.dae"/>
@@ -47,7 +47,7 @@
         <parent link="base"/>
         <child link="handle"/>
-        <origin xyz="0 0 0" rpy="0 0 0"/>
-        <axis xyz="0 1 0"/>
-        <dynamics damping="0.0" friction="10.0" />
+        <origin xyz="0 0 0.071" rpy="0 0 0"/> <!-- 0.071 -->
+        <axis xyz="0 0 1"/>
+        <dynamics damping="0.0" friction="0.01" />
         <limit effort="100" velocity="0.5" />
     </joint>
@@ -58,5 +58,4 @@
         </joint>
         <actuator name="needle_valve_actuator">
-            <hardwareInterface>hardware_interface/EffortJointInterface</hardwareInterface>
             <mechanicalReduction>1</mechanicalReduction>
         </actuator>
@@ -65,11 +64,11 @@
     <link name="handle">
         <collision>
-            <origin xyz="0 0 0" rpy="0 0 0"/>
+            <origin xyz="0 0 0" rpy="0 -1.5708 0"/>
             <geometry>
-                <mesh filename="package://manipulation_playground_articulated_devices/devices/needle_valve/model/needle_valve_handle.dae"/>
+                <cylinder radius="0.0063" length="0.055"/>
             </geometry>
         </collision>
         <visual>
-            <origin xyz="0 0 0" rpy="0 0 0"/>
+            <origin xyz="0 0 -0.071" rpy="-1.5708 0 -1.5708"/>
             <geometry>
                 <mesh filename="package://manipulation_playground_articulated_devices/devices/needle_valve/model/needle_valve_handle.dae"/>
@@ -81,6 +80,6 @@
             <inertia
                 ixx="${mass2 / 12.0 * (3.0*radius2*radius2 + length2*length2)}" ixy="0.0" ixz="0.0"
-                iyy="${mass2 / 2.0 * (radius2*radius2)}" iyz="0.0"
-                izz="${mass2 / 12.0 * (3.0*radius2*radius2 + length2*length2)}"/>
+                iyy="${mass2 / 12.0 * (3.0*radius2*radius2 + length2*length2)}" iyz="0.0"
+                izz="${mass2 / 2.0 * (radius2*radius2)}"/>
         </inertial>
     </link>

Commit message: Added ability to toggle continuous joint when loading needle valve

File: manipulation_playground_articulated_devices/devices/needle_valve/model/needle_valve.urdf.xacro (robot description, xacro)
@@ -2,100 +2,116 @@
 <!-- Interactable Needle Valve -->
 <robot name="needle_valve" xmlns:xacro="http://www.ros.org/wiki/xacro">
-    <!-- Dimensions for Inertias -->
-    <!-- Base -->
-    <xacro:property name="width1" value="0.5"/>
-    <xacro:property name="height1" value="0.1"/>
-    <xacro:property name="mass1" value="0.5"/>
-    <!-- Handle -->
-    <xacro:property name="length2" value="0.01"/>
-    <xacro:property name="radius2" value="0.03"/>
-    <xacro:property name="mass2" value="1"/>
-    <!-- Import all Gazebo-customization elements -->
-    <xacro:include filename="$(find manipulation_playground_articulated_devices)/devices/needle_valve/model/needle_valve.gazebo" />
-    <!-- Used to fix switch to world -->
-    <link name="world"/>
-    <joint name="needle_valve_base_to_world" type="fixed">
-        <parent link="world"/>
-        <child link="base"/>
-        <origin xyz="0 0 0" rpy="0 0 0"/>
-    </joint>
-    <!-- Needle Valve Base -->
-    <link name="base">
-        <collision>
-            <origin xyz="0 0 0.01" rpy="-1.5708 0 -1.5708"/>
-            <geometry>
-                <box size="0.065 0.05 0.03"/>
-            </geometry>
-        </collision>
-        <visual>
-            <origin xyz="0 0 0" rpy="-1.5708 0 -1.5708"/>
-            <geometry>
-                <mesh filename="package://manipulation_playground_articulated_devices/devices/needle_valve/model/needle_valve_base.dae"/>
-            </geometry>
-        </visual>
-        <inertial>
-            <origin xyz="0 0 ${height1/2}" rpy="0 0 0"/>
-            <mass value="${mass1}"/>
-            <inertia
-                ixx="${mass1 / 12.0 * (width1*width1 + height1*height1)}" ixy="0.0" ixz="0.0"
-                iyy="${mass1 / 12.0 * (height1*height1 + width1*width1)}" iyz="0.0"
-                izz="${mass1 / 12.0 * (width1*width1 + width1*width1)}"/>
-        </inertial>
-    </link>
-    <joint name="needle_valve_handle_to_base" type="fixed">
-        <parent link="base"/>
-        <child link="handle"/>
-        <origin xyz="0 0 0.071" rpy="0 0 0"/>
-    </joint>
-    <link name="handle">
-        <inertial>
-            <origin xyz="0 0 0" rpy="0 0 0" />
-            <mass value="1" />
-            <inertia
-            ixx="1.0" ixy="0.0" ixz="0.0"
-            iyy="1.0" iyz="0.0"
-            izz="1.0" />
-        </inertial>
-    </link>
-    <!-- Needle Valve Joint -->
-    <joint name="needle_valve_joint" type="continuous">
-        <parent link="handle"/>
-        <child link="handle_rotated"/>
-        <origin xyz="0 0 0" rpy="0 0 0"/>
-        <axis xyz="0 0 1"/>
-        <dynamics damping="0.0" friction="0.01" />
-        <limit effort="100" velocity="0.5" />
-    </joint>
-    <transmission name="needle_valve_trans">
-        <type>transmission_interface/SimpleTransmission</type>
-        <joint name="needle_valve_joint">
-            <hardwareInterface>hardware_interface/EffortJointInterface</hardwareInterface>
+    <xacro:arg name="continuous" default="true"/>
+    <xacro:macro name="needle_valve" params="continuous:=true">
+        <!-- Dimensions for Inertias -->
+        <!-- Base -->
+        <xacro:property name="width1" value="0.5"/>
+        <xacro:property name="height1" value="0.1"/>
+        <xacro:property name="mass1" value="0.5"/>
+        <!-- Handle -->
+        <xacro:property name="length2" value="0.01"/>
+        <xacro:property name="radius2" value="0.03"/>
+        <xacro:property name="mass2" value="1"/>
+        <!-- Import all Gazebo-customization elements -->
+        <xacro:include filename="$(find manipulation_playground_articulated_devices)/devices/needle_valve/model/needle_valve.gazebo" />
+        <!-- Used to fix switch to world -->
+        <link name="world"/>
+        <joint name="needle_valve_base_to_world" type="fixed">
+            <parent link="world"/>
+            <child link="base"/>
+            <origin xyz="0 0 0" rpy="0 0 0"/>
         </joint>
-        <actuator name="needle_valve_actuator">
-            <mechanicalReduction>1</mechanicalReduction>
-        </actuator>
-    </transmission>
-    <!-- Needle Valve Handle -->
-    <link name="handle_rotated">
-        <collision>
-            <origin xyz="0 0 0" rpy="0 -1.5708 1.5708"/>
-            <geometry>
-                <cylinder radius="0.0063" length="0.055"/>
-            </geometry>
-        </collision>
-        <visual>
-            <origin xyz="0 0 -0.071" rpy="-1.5708 0 0"/>
-            <geometry>
-                <mesh filename="package://manipulation_playground_articulated_devices/devices/needle_valve/model/needle_valve_handle.dae"/>
-            </geometry>
-        </visual>
-        <inertial>
-            <origin xyz="0 0 0" rpy="0 0 0"/>
-            <mass value="${mass2}"/>
-            <inertia
-                ixx="${mass2 / 12.0 * (3.0*radius2*radius2 + length2*length2)}" ixy="0.0" ixz="0.0"
-                iyy="${mass2 / 12.0 * (3.0*radius2*radius2 + length2*length2)}" iyz="0.0"
-                izz="${mass2 / 2.0 * (radius2*radius2)}"/>
-        </inertial>
-    </link>
+        <!-- Needle Valve Base -->
+        <link name="base">
+            <collision>
+                <origin xyz="0 0 0.01" rpy="-1.5708 0 -1.5708"/>
+                <geometry>
+                    <box size="0.065 0.05 0.03"/>
+                </geometry>
+            </collision>
+            <visual>
+                <origin xyz="0 0 0" rpy="-1.5708 0 -1.5708"/>
+                <geometry>
+                    <mesh filename="package://manipulation_playground_articulated_devices/devices/needle_valve/model/needle_valve_base.dae"/>
+                </geometry>
+            </visual>
+            <inertial>
+                <origin xyz="0 0 ${height1/2}" rpy="0 0 0"/>
+                <mass value="${mass1}"/>
+                <inertia
+                    ixx="${mass1 / 12.0 * (width1*width1 + height1*height1)}" ixy="0.0" ixz="0.0"
+                    iyy="${mass1 / 12.0 * (height1*height1 + width1*width1)}" iyz="0.0"
+                    izz="${mass1 / 12.0 * (width1*width1 + width1*width1)}"/>
+            </inertial>
+        </link>
+        <joint name="needle_valve_handle_to_base" type="fixed">
+            <parent link="base"/>
+            <child link="handle"/>
+            <origin xyz="0 0 0.071" rpy="0 0 0"/>
+        </joint>
+        <link name="handle">
+            <inertial>
+                <origin xyz="0 0 0" rpy="0 0 0" />
+                <mass value="1" />
+                <inertia
+                ixx="1.0" ixy="0.0" ixz="0.0"
+                iyy="1.0" iyz="0.0"
+                izz="1.0" />
+            </inertial>
+        </link>
+        <!-- Needle Valve Joint -->
+        <xacro:if value="${continuous}">
+            <joint name="needle_valve_joint" type="continuous">
+                <parent link="handle"/>
+                <child link="handle_rotated"/>
+                <origin xyz="0 0 0" rpy="0 0 0"/>
+                <axis xyz="0 0 1"/>
+                <dynamics damping="0.0" friction="0.01" />
+                <limit effort="100" velocity="0.5" />
+            </joint>
+        </xacro:if>
+        <xacro:unless value="${continuous}">
+            <joint name="needle_valve_joint" type="revolute">
+                <parent link="handle"/>
+                <child link="handle_rotated"/>
+                <origin xyz="0 0 0" rpy="0 0 0"/>
+                <axis xyz="0 0 1"/>
+                <dynamics damping="0.0" friction="0.01" />
+                <limit effort="100" lower="-3.0" upper="3.0" velocity="0.5" />
+            </joint>
+        </xacro:unless>
+        <transmission name="needle_valve_trans">
+            <type>transmission_interface/SimpleTransmission</type>
+            <joint name="needle_valve_joint">
+                <hardwareInterface>hardware_interface/EffortJointInterface</hardwareInterface>
+            </joint>
+            <actuator name="needle_valve_actuator">
+                <mechanicalReduction>1</mechanicalReduction>
+            </actuator>
+        </transmission>
+        <!-- Needle Valve Handle -->
+        <link name="handle_rotated">
+            <collision>
+                <origin xyz="0 0 0" rpy="0 -1.5708 1.5708"/>
+                <geometry>
+                    <cylinder radius="0.0063" length="0.055"/>
+                </geometry>
+            </collision>
+            <visual>
+                <origin xyz="0 0 -0.071" rpy="-1.5708 0 0"/>
+                <geometry>
+                    <mesh filename="package://manipulation_playground_articulated_devices/devices/needle_valve/model/needle_valve_handle.dae"/>
+                </geometry>
+            </visual>
+            <inertial>
+                <origin xyz="0 0 0" rpy="0 0 0"/>
+                <mass value="${mass2}"/>
+                <inertia
+                    ixx="${mass2 / 12.0 * (3.0*radius2*radius2 + length2*length2)}" ixy="0.0" ixz="0.0"
+                    iyy="${mass2 / 12.0 * (3.0*radius2*radius2 + length2*length2)}" iyz="0.0"
+                    izz="${mass2 / 2.0 * (radius2*radius2)}"/>
+            </inertial>
+        </link>
+    </xacro:macro>
+    <xacro:needle_valve continuous="$(arg continuous)"/>
 </robot>

Commit message: Added 'very stiff' dynamics mode for needle_valve.

File: manipulation_playground_articulated_devices/devices/needle_valve/model/needle_valve.urdf.xacro (robot description, xacro)
@@ -79,4 +79,5 @@
                 <dynamics damping="0.0" friction="0.01" />
                 <limit effort="100" lower="-3.0" upper="3.0" velocity="0.5" />
+                <!-- <limit effort="100" lower="-0.7854" upper="0.7854" velocity="0.5" /> -->
             </joint>
         </xacro:unless>
